Commit message: Adding maths example for xacro

File: xacro_demo.xacro (robot description, xacro)
@@ -1,6 +1,8 @@
 <?xml version="1.0"?>
-<robot xmlns:xacro="http://www.ros.org/wiki/xacro" name="firefighter">
+<robot xmlns:xacro="http://www.ros.org/wiki/xacro" name="r2d2">
 <xacro:property name="width" value="0.2" />
 <xacro:property name="bodylen" value="0.6" />
+<xacro:property name="wheeldiam" value="0.1" />
+<xacro:property name="reflect" value="0.9" />
 <link name="base_link">
     <visual>
@@ -16,3 +18,11 @@
     </collision>
 </link>
+<link name="wheel">
+    <visual>
+        <geometry>
+            <cylinder radius="${wheeldiam/2}" length="0.1"/>
+        </geometry>
+        <origin xyz="${reflect*(width+.02)} 0 0.25" />
+    </visual>
+</link>
 </robot>

Commit message: Adding macro to my xacro example

File: xacro_demo.xacro (robot description, xacro)
@@ -5,4 +5,12 @@
 <xacro:property name="wheeldiam" value="0.1" />
 <xacro:property name="reflect" value="0.9" />
+<xacro:macro name="default_inertial" params="mass">
+    <inertial>
+            <mass value="${mass}" />
+            <inertia ixx="1.0" ixy="0.0" ixz="0.0"
+                 iyy="1.0" iyz="0.0"
+                 izz="1.0" />
+    </inertial>
+</xacro:macro>
 <link name="base_link">
     <visual>
@@ -17,4 +25,5 @@
         </geometry>
     </collision>
+    <xacro:default_inertial mass="10"/>
 </link>
 <link name="wheel">

Commit message: More advanced macro for my xacro example.

File: xacro_demo.xacro (robot description, xacro)
@@ -12,4 +12,19 @@
                  izz="1.0" />
     </inertial>
+</xacro:macro>
+<xacro:macro name="blue_shape" params="name *shape">
+    <link name="${name}">
+        <visual>
+            <geometry>
+                <xacro:insert_block name="shape" />
+            </geometry>
+            <material name="blue"/>
+        </visual>
+        <collision>
+            <geometry>
+                <xacro:insert_block name="shape" />
+            </geometry>
+        </collision>
+    </link>
 </xacro:macro>
 <link name="base_link">
@@ -35,3 +50,6 @@
     </visual>
 </link>
+<xacro:blue_shape name="blue_cylinder">
+    <cylinder radius=".42" length=".01" />
+</xacro:blue_shape>
 </robot>
